File: mp3_player.kicad_pcb (KiCad board)
At the start: 2 copper layers, 67 x 97.5 mm, 13 parts, among them J1 AudioJack3_SwitchTR, SW1 Power, SW2 Pause/Play, SW3 Next, SW4 Previous/Restart, SW5 Seek Forward / Backward, SW6 Volume Up, SW7 Volume Down

Commit message: Finish up PCB and send to manufacturer
Parts:
- added J2: Conn_01x02, Connector_JST:JST_PH_S2B-PH-K_1x02_P2.00mm_Horizontal, B.Cu at (170.0, 95.5)
- added REF**: MountingHole_2.1mm, MountingHole:MountingHole_2.1mm, F.Cu at (170.5, 53.0)
- added REF**: MountingHole_2.1mm, MountingHole:MountingHole_2.1mm, F.Cu at (110.0, 53.0)
- added REF**: MountingHole_2.1mm, MountingHole:MountingHole_2.1mm, F.Cu at (110.5, 143.5)
- added REF**: MountingHole_2.1mm, MountingHole:MountingHole_2.1mm, F.Cu at (169.0, 130.0)
- SW6, SW7: footprint Button_Switch_THT:SW_PUSH_6mm -> Button_Switch_THT:SW_Tactile_SPST_Angled_PTS645Vx39-2LFS
- moved SW6 57.2 mm to (171.0, 69.5), turned to -90 degrees
- moved SW7 56.8 mm to (171.0, 80.0), turned to -90 degrees
- moved J1 53.3 mm to (166.2, 142.3)
- moved SW2 53.3 mm to (136.7, 136.3)
- moved SW4 53.3 mm to (148.7, 136.3)
- moved U1 53.3 mm to (128.7, 74.3)
- moved U11 53.3 mm to (141.7, 65.5)
- moved U2 53.3 mm to (145.1, 117.5)
- moved A1 53.3 mm to (118.7, 102.4)
- moved SW1 53.3 mm to (121.7, 52.8)
- moved SW3 53.3 mm to (124.7, 136.3)
- moved SW5 53.3 mm to (109.7, 80.3)
- moved U3 53.3 mm to (172.6, 62.1)
Connections:
- A1 pad 30: 3.7V -> Net-(A1-VIN)
- SW1 pad 1: unconnected-(SW1-A-Pad1) -> 3.7V
- SW1 pad 2: unconnected-(SW1-B-Pad2) -> Net-(A1-VIN)
- U11 pad 4: unconnected-(U11-BAT--Pad4) -> Net-(J2-Pin_1)
- U11 pad 6: unconnected-(U11-BAT+-Pad6) -> Net-(J2-Pin_2)
Routing:
- net VOLDN: track 61.1 -> 154.7 mm
- net Net-(A1-VIN): track 0.00 -> 44.4 mm
- net Net-(J2-Pin_2): track 0.00 -> 43.5 mm
- net Net-(J2-Pin_1): track 0.00 -> 30.6 mm
- net 3.7V: track 63.8 -> 79.1 mm
- net VOLUP: track 70.8 -> 73.9 mm
- net GND: track 206.4 -> 203.3 mm
Other:
- outline, holes or cut-outs redrawn
